Commit message: fix: estimate C049 simulation limits from speed and gear ratios

File: simulation/urdf/so_arm_102.urdf (robot description, URDF)
Before this commit: robot so_arm_102_pre_for_urdf_v5, 8 links, 7 joints
Joints:
- joint clamp1: limit lower=0 upper=0.0415 effort=408.6 velocity=0.0340 -> lower=0 upper=0.0415 effort=226.2 velocity=0.0562
- joint clamp2: limit lower=-0.0415 upper=3.46944695195e-17 effort=408.6 velocity=0.0340 -> lower=-0.0415 upper=3.46944695195e-17 effort=226.2 velocity=0.0562
- joint link4_to_link5: limit lower=-2.87979326579 upper=2.84488668075 effort=2.942 velocity=4.717 -> lower=-2.87979326579 upper=2.84488668075 effort=1.629 velocity=7.808

File: simulation/urdf/so_arm_102.xacro (robot description, xacro)
@@ -5230,8 +5230,22 @@
     <limit effort="2.942" velocity="4.717" lower="-1.72787595947" upper="1.69296937443" />
   </joint>
-  <!-- Hardware: ST-3215-C049, 12 V, 1:191 (see docs/bom.md).
-       TODO: replace effort and velocity after confirming the C049 datasheet.
-       Current values are retained from PR #21: C018, 1:345 assumptions,
-       NOT verified C049 limits or continuous operating ratings. -->
+  <!-- C049 simulation estimates, NOT manufacturer specifications or hardware settings.
+       Hardware: ST-3215-C049, 12 V, 1:191 (docs/bom.md).
+       C018 reference at 12 V from PR #21: 30 kg.cm stall, 0.222 s/60 deg.
+       Speed estimate using the 7.4 V C001/C044 comparison:
+         0.222 * (0.116 / 0.192) = 0.134125 s/60 deg = 7.807624 rad/s.
+       Torque estimate assumes the C018 motor/current limit and gearbox efficiency:
+         30 * (191 / 345) = 16.608696 kg.cm stall = 1.628757 N.m.
+       The two estimates use different approximations; they are not a measured curve.
+       The 7.4 V variants differ in motor/current characteristics, so do not scale
+       their torque ratings onto C049. Continuous torque is not established here.
+       Jaw limits retain PR #21's convention: torque / 0.0072 m and speed * 0.0072 m.
+       The mimic jaw is not a second independent motor or an extra torque budget.
+       Replace these estimates after obtaining a C049 datasheet or bench measurements.
+       Sources:
+       https://github.com/roboninecom/SO-ARM102/pull/21
+       https://files.seeedstudio.com/products/Feetech/108090023_STS3215-C001_Datasheet.pdf
+       https://files.seeedstudio.com/products/Feetech/101090141_Feetech_ST-3215-C044_Datasheet.pdf
+  -->
   <joint name="link4_to_link5" type="revolute">
     <origin xyz="0.0591945817497 -0.0180002669618 -4.03637807994e-05" rpy="0 0 0" />
@@ -5239,10 +5253,7 @@
     <child link="link5_1" />
     <axis xyz="-1 -4.90398764451e-08 1.40482066922e-10" />
-    <limit effort="2.942" velocity="4.717" lower="-2.87979326579" upper="2.84488668075" />
+    <limit effort="1.629" velocity="7.808" lower="-2.87979326579" upper="2.84488668075" />
   </joint>
-  <!-- Hardware: ST-3215-C049, 12 V, 1:191 (see docs/bom.md).
-       TODO: replace effort and velocity after confirming the C049 datasheet.
-       Current values are retained from PR #21: C018, 1:345 assumptions,
-       NOT verified C049 limits or continuous operating ratings. -->
+  <!-- Estimated C049 limits; see the calculation above link4_to_link5. -->
   <joint name="clamp1" type="prismatic">
     <origin xyz="0.0639999993385 0.0165020797222 0.0159979235363" rpy="0 0 0" />
@@ -5250,10 +5261,7 @@
     <child link="clamp1_1" />
     <axis xyz="-5.21612507542e-08 1 4.50838078172e-08" />
-    <limit effort="408.6" velocity="0.0340" lower="0" upper="0.0415" />
+    <limit effort="226.2" velocity="0.0562" lower="0" upper="0.0415" />
   </joint>
-  <!-- Hardware: ST-3215-C049, 12 V, 1:191 (see docs/bom.md).
-       TODO: replace effort and velocity after confirming the C049 datasheet.
-       Current values are retained from PR #21: C018, 1:345 assumptions,
-       NOT verified C049 limits or continuous operating ratings. -->
+  <!-- Estimated C049 limits; see the calculation above link4_to_link5. -->
   <joint name="clamp2" type="prismatic">
     <origin xyz="0.0640000007627 -0.0154979202778 0.0159979219163" rpy="0 0 0" />
@@ -5261,5 +5269,5 @@
     <child link="clamp2_1" />
     <axis xyz="-4.9039873492e-08 1 4.73420869362e-08" />
-    <limit effort="408.6" velocity="0.0340" lower="-0.0415" upper="3.46944695195e-17" />
+    <limit effort="226.2" velocity="0.0562" lower="-0.0415" upper="3.46944695195e-17" />
     <mimic joint="clamp1" multiplier="-1" offset="0" />
   </joint>
